File: Micro Data Logger/Micro Data Logger.sch (KiCad schematic (older format))
At the start: 2 parts

Commit message: Added more devices
Parts:
- removed U?: ATXMEGA32E5-MU, VQFN32, symbol atmel:ATXMEGA32E5-MU
- added C? (x2): 10uF, symbol device:C
- added C?: 47uF, symbol device:C
- added D? (x2): LED, symbol device:LED
- added J?: Conn_01x02, symbol Connector:Conn_01x02
- added R? (x2): 100, symbol device:R
- added SW?: SW_DIP_x10, symbol Switch:SW_DIP_x10
- added SW?: SW_SPDT, symbol Switch:SW_SPDT
- added SW?: SW_DIP_x04, symbol Switch:SW_DIP_x04
- added U?: LMT86DCK, TO_SOT_Packages_SMD:SOT-353_SC-70-5, symbol sensors:LMT86DCK
- added U? (x2): MAX31856, Housings_SSOP:TSSOP-14_4.4x5mm_Pitch0.65mm, symbol sensors:MAX31856
- added U?: ADS1234IPW, symbol adc-dac:ADS1234IPW
- added U?: MCP1700-3302E_SOT23, TO_SOT_Packages_SMD:SOT-23, symbol regul:MCP1700-3302E_SOT23
- added U?: ATMEGA644PA-MU, VQFN44, symbol atmel:ATMEGA644PA-MU
- added Y?: Crystal, symbol device:Crystal
Connections:
- net labels added: +3.3V, +5V, GND, GNDA
- wire segments 0 -> 28
Other:
- moved on the sheet: J?

Commit message: Changed Voltage Regulator
Parts:
- removed U?: MCP1700-3302E_SOT23, TO_SOT_Packages_SMD:SOT-23, symbol regul:MCP1700-3302E_SOT23
- added U?: MIC5219-3.3, TO_SOT_Packages_SMD:SOT-23-5, symbol regul:MIC5219-3.3
Connections:
- wire segments 28 -> 27
Changed lines of the file:
@@
-$EndComp
-$Comp
-L regul:MCP1700-3302E_SOT23 U?
-U 1 1 5A84FBCC
-P 6500 900
-F 0 "U?" H 6500 1142 50  0000 C CNN
-F 1 "MCP1700-3302E_SOT23" H 6500 1051 50  0000 C CNN
-F 2 "TO_SOT_Packages_SMD:SOT-23" H 6500 1125 50  0001 C CNN
-F 3 "http://ww1.microchip.com/downloads/en/DeviceDoc/20001826C.pdf" H 6500 900 50  0001 C CNN
-	1    6500 900
-	1    0    0    -1
 $EndComp
 $Comp
@@
 	6900 1200 7400 1200
 Connection ~ 6900 1200
-Wire Wire Line
-	6500 1200 6900 1200
-Connection ~ 6500 1200
 Connection ~ 5950 900
 Connection ~ 5950 1200
@@
 	1    0    0    -1
 $EndComp
-Wire Wire Line
-	5950 1200 6500 1200
 $Comp
 L atmel:ATMEGA644PA-MU U?
@@
 	0    1    1    0
 $EndComp
+Wire Wire Line
+	5950 1200 6900 1200
+$Comp
+L regul:MIC5219-3.3 U?
+U 1 1 5A86A15C
+P 6500 700
+F 0 "U?" H 6500 1042 50  0000 C CNN
+F 1 "MIC5219-3.3" H 6500 951 50  0000 C CNN
+F 2 "TO_SOT_Packages_SMD:SOT-23-5" H 6500 1025 50  0001 C CNN
+F 3 "http://ww1.microchip.com/downloads/en/devicedoc/mic5219.pdf" H 6500 700 50  0001 C CNN
+	1    6500 700
+	1    0    0    -1
+$EndComp
 $EndSCHEMATC
